File: supercap_dev.kicad_pcb (KiCad board)
At the start: 2 copper layers, 92.1 x 34.5 mm, 32 parts, among them J1 Conn_01x02_Socket, J2 Conn_01x02_Socket, J4 Conn_01x02_Socket, Q1 WST3325, Q5 SS8550, Q6 SS8550

Commit message: Done
Other:
- board size 92.1 x 34.5 mm -> 92.1 x 34.3 mm
